File: quad_analog_pullup.kicad_sch (KiCad schematic)
At the start: 25 parts, among them U1101 MCP6004, U4 SRV05-4

Commit message: Started moving to pin headers
Connections:
- net +5V: now also U1101.4 (V+)
- net GND: now also U1101.11 (V-)
- net at C16.1, RN1101.5 (R4.2), U4.4 (IO3): now also U1101.12 (+); no longer U1101.3 (+)
- net at C15.1, RN1101.6 (R3.2), U4.3 (IO2): now also U1101.10 (+); no longer U1101.3 (+)
- net at C14.1, RN1101.7 (R2.2), U4.1 (IO1): now also U1101.5 (+); no longer U1101.3 (+)
- new net: R26.2, U1101.6 (-), U1101.7
- new net: R27.2, U1101.8, U1101.9 (-)
- new net: R28.2, U1101.13 (-), U1101.14
Changed lines of the file:
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@@
     (effects (font (size 1.27 1.27)) (justify right))
   )
-  (symbol (lib_id "Amplifier_Operational:MCP6004") (at 41.275 42.545 0)
+  (symbol (lib_id "Amplifier_Operational:MCP6004") (at 41.275 42.545 0) (unit 5)
     (in_bom yes) (on_board yes)
     (property "Reference" "U1101" (id 0) (at 40.2082 41.3766 0)
@@
     (pin "4")
   )
-  (symbol (lib_id "Device:R_Pack04") (at 78.74 92.075 270)
+  (symbol (lib_id "Device:R_Pack04") (at 78.74 92.075 270) (unit 1)
     (in_bom yes) (on_board yes)
     (property "Reference" "RN1101" (id 0) (at 78.74 81.4832 90))
@@
     (pin "8")
   )
-  (symbol (lib_id "Device:R") (at 45.72 77.47 0)
+  (symbol (lib_id "Device:R") (at 45.72 77.47 0) (unit 1)
     (in_bom yes) (on_board yes)
     (property "Reference" "R1101" (id 0) (at 47.498 76.3016 0)
@@
     (pin "2")
   )
-  (symbol (lib_id "Device:C") (at 29.845 42.545 0)
+  (symbol (lib_id "Device:C") (at 29.845 42.545 0) (unit 1)
     (in_bom yes) (on_board yes)
     (property "Reference" "C1101" (id 0) (at 32.766 41.3766 0)
@@
     (pin "2")
   )
-  (symbol (lib_id "power:GND") (at 38.735 52.705 0)
+  (symbol (lib_id "power:GND") (at 38.735 52.705 0) (unit 1)
     (in_bom yes) (on_board yes)
     (property "Reference" "#PWR01102" (id 0) (at 38.735 59.055 0)
@@
     (pin "1")
   )
-  (symbol (lib_id "power:GND") (at 106.68 104.775 0)
+  (symbol (lib_id "power:GND") (at 106.68 104.775 0) (unit 1)
     (in_bom yes) (on_board yes)
     (property "Reference" "#PWR01108" (id 0) (at 106.68 111.125 0)
@@
     (pin "1")
   )
-  (symbol (lib_id "power:GND") (at 116.84 104.775 0)
+  (symbol (lib_id "power:GND") (at 116.84 104.775 0) (unit 1)
     (in_bom yes) (on_board yes)
     (property "Reference" "#PWR01109" (id 0) (at 116.84 111.125 0)
@@
     (pin "1")
   )
-  (symbol (lib_id "power:GND") (at 217.805 97.79 0)
+  (symbol (lib_id "power:GND") (at 217.805 97.79 0) (unit 1)
     (in_bom yes) (on_board yes)
     (property "Reference" "#PWR01105" (id 0) (at 217.805 104.14 0)
@@
     (pin "1")
   )
-  (symbol (lib_id "Device:C") (at 45.72 64.77 0)
+  (symbol (lib_id "Device:C") (at 45.72 64.77 0) (unit 1)
     (in_bom yes) (on_board yes)
     (property "Reference" "C1409" (id 0) (at 48.641 63.6016 0)
@@
     (pin "2")
   )
-  (symbol (lib_id "power:GND") (at 45.72 60.96 180)
+  (symbol (lib_id "power:GND") (at 45.72 60.96 180) (unit 1)
     (in_bom yes) (on_board yes)
     (property "Reference" "#PWR0210" (id 0) (at 45.72 54.61 0)
@@
     (pin "1")
   )
-  (symbol (lib_id "Device:R") (at 54.61 77.47 0)
+  (symbol (lib_id "Device:R") (at 54.61 77.47 0) (unit 1)
     (in_bom yes) (on_board yes)
     (property "Reference" "R1102" (id 0) (at 56.388 76.3016 0)
@@
     (pin "2")
   )
-  (symbol (lib_id "Device:R") (at 62.865 77.47 0)
+  (symbol (lib_id "Device:R") (at 62.865 77.47 0) (unit 1)
     (in_bom yes) (on_board yes)
     (property "Reference" "R1103" (id 0) (at 64.643 76.3016 0)
@@
     (pin "2")
   )
-  (symbol (lib_id "Device:R") (at 71.12 77.47 0)
+  (symbol (lib_id "Device:R") (at 71.12 77.47 0) (unit 1)
     (in_bom yes) (on_board yes)
     (property "Reference" "R1104" (id 0) (at 72.898 76.3016 0)
@@
     (pin "2")
   )
-  (symbol (lib_id "Amplifier_Operational:MCP6004") (at 172.72 68.58 0)
+  (symbol (lib_id "Amplifier_Operational:MCP6004") (at 172.72 68.58 0) (unit 1)
     (in_bom yes) (on_board yes)
     (property "Reference" "U1101" (id 0) (at 172.72 59.2582 0))
@@
     (pin "3")
   )
-  (symbol (lib_id "Amplifier_Operational:MCP6004") (at 172.72 83.185 0)
+  (symbol (lib_id "Amplifier_Operational:MCP6004") (at 172.72 83.185 0) (unit 2)
     (in_bom yes) (on_board yes)
     (property "Reference" "U1101" (id 0) (at 172.72 73.8632 0))
@@
     (pin "7")
   )
-  (symbol (lib_id "Amplifier_Operational:MCP6004") (at 172.72 97.79 0)
+  (symbol (lib_id "Amplifier_Operational:MCP6004") (at 172.72 97.79 0) (unit 3)
     (in_bom yes) (on_board yes)
     (property "Reference" "U1101" (id 0) (at 172.72 88.4682 0))
@@
     (pin "9")
   )
-  (symbol (lib_id "Amplifier_Operational:MCP6004") (at 172.72 112.395 0)
+  (symbol (lib_id "Amplifier_Operational:MCP6004") (at 172.72 112.395 0) (unit 4)
     (in_bom yes) (on_board yes)
     (property "Reference" "U1101" (id 0) (at 172.72 103.0732 0))
@@
     (pin "14")
   )
-  (symbol (lib_id "power:GND") (at 86.36 104.775 0)
+  (symbol (lib_id "power:GND") (at 86.36 104.775 0) (unit 1)
     (in_bom yes) (on_board yes)
     (property "Reference" "#PWR01106" (id 0) (at 86.36 111.125 0)
@@
     (pin "1")
   )
-  (symbol (lib_id "power:GND") (at 96.52 104.775 0)
+  (symbol (lib_id "power:GND") (at 96.52 104.775 0) (unit 1)
     (in_bom yes) (on_board yes)
     (property "Reference" "#PWR01107" (id 0) (at 96.52 111.125 0)
@@
     (pin "6")
   )
-  (symbol (lib_id "power:GND") (at 128.905 78.74 0)
+  (symbol (lib_id "power:GND") (at 128.905 78.74 0) (unit 1)
     (in_bom yes) (on_board yes)
     (property "Reference" "#PWR0272" (id 0) (at 128.905 85.09 0)
