File: lowside_quad.kicad_sch (KiCad schematic)
At the start: 4 parts, among them U401 VNLD5160, U402 VNLD5160

Commit message: Started moving to pin headers
Parts:
- renumbered RN401 to RN301, RN402 to RN302, U401 to U301, U402 to U302
Changed lines of the file:
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@@
   (symbol (lib_id "vnld5090:VNLD5090") (at 106.045 51.435 0)
     (in_bom yes) (on_board yes)
-    (property "Reference" "U401" (id 0) (at 106.045 35.0012 0)
+    (property "Reference" "U301" (id 0) (at 106.045 35.0012 0)
       (effects (font (size 1.524 1.524)))
     )
@@
   (symbol (lib_id "vnld5090:VNLD5090") (at 106.045 93.345 0)
     (in_bom yes) (on_board yes)
-    (property "Reference" "U402" (id 0) (at 106.045 76.9112 0)
+    (property "Reference" "U302" (id 0) (at 106.045 76.9112 0)
       (effects (font (size 1.524 1.524)))
     )
@@
   (symbol (lib_id "Device:R_Pack04") (at 78.105 71.12 270) (mirror x)
     (in_bom yes) (on_board yes)
-    (property "Reference" "RN401" (id 0) (at 78.105 81.7118 90))
+    (property "Reference" "RN301" (id 0) (at 78.105 81.7118 90))
     (property "Value" "1k" (id 1) (at 78.105 79.4004 90))
     (property "Footprint" "Resistor_SMD:R_Array_Convex_4x0603" (id 2) (at 78.105 64.135 90)
@@
   (symbol (lib_id "Device:R_Pack04") (at 67.945 83.82 0)
     (in_bom yes) (on_board yes)
-    (property "Reference" "RN402" (id 0) (at 57.3532 83.82 90))
+    (property "Reference" "RN302" (id 0) (at 57.3532 83.82 90))
     (property "Value" "1k" (id 1) (at 59.6646 83.82 90))
     (property "Footprint" "Resistor_SMD:R_Array_Convex_4x0603" (id 2) (at 74.93 83.82 90)

Commit message: Right hand pinout completed
Parts:
- renumbered RN301 to RN501, RN302 to RN502, U301 to U501, U302 to U502
Changed lines of the file:
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@@
   (symbol (lib_id "vnld5090:VNLD5090") (at 106.045 51.435 0)
     (in_bom yes) (on_board yes)
-    (property "Reference" "U301" (id 0) (at 106.045 35.0012 0)
+    (property "Reference" "U501" (id 0) (at 106.045 35.0012 0)
       (effects (font (size 1.524 1.524)))
     )
@@
   (symbol (lib_id "vnld5090:VNLD5090") (at 106.045 93.345 0)
     (in_bom yes) (on_board yes)
-    (property "Reference" "U302" (id 0) (at 106.045 76.9112 0)
+    (property "Reference" "U502" (id 0) (at 106.045 76.9112 0)
       (effects (font (size 1.524 1.524)))
     )
@@
   (symbol (lib_id "Device:R_Pack04") (at 78.105 71.12 270) (mirror x)
     (in_bom yes) (on_board yes)
-    (property "Reference" "RN301" (id 0) (at 78.105 81.7118 90))
+    (property "Reference" "RN501" (id 0) (at 78.105 81.7118 90))
     (property "Value" "1k" (id 1) (at 78.105 79.4004 90))
     (property "Footprint" "Resistor_SMD:R_Array_Convex_4x0603" (id 2) (at 78.105 64.135 90)
@@
   (symbol (lib_id "Device:R_Pack04") (at 67.945 83.82 0)
     (in_bom yes) (on_board yes)
-    (property "Reference" "RN302" (id 0) (at 57.3532 83.82 90))
+    (property "Reference" "RN502" (id 0) (at 57.3532 83.82 90))
     (property "Value" "1k" (id 1) (at 59.6646 83.82 90))
     (property "Footprint" "Resistor_SMD:R_Array_Convex_4x0603" (id 2) (at 74.93 83.82 90)

Commit message: Started left hand side
Parts:
- renumbered RN501 to RN201, RN502 to RN202, U501 to U201, U502 to U202
Changed lines of the file:
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@@
   (symbol (lib_id "vnld5090:VNLD5090") (at 106.045 51.435 0)
     (in_bom yes) (on_board yes)
-    (property "Reference" "U501" (id 0) (at 106.045 35.0012 0)
+    (property "Reference" "U201" (id 0) (at 106.045 35.0012 0)
       (effects (font (size 1.524 1.524)))
     )
@@
   (symbol (lib_id "vnld5090:VNLD5090") (at 106.045 93.345 0)
     (in_bom yes) (on_board yes)
-    (property "Reference" "U502" (id 0) (at 106.045 76.9112 0)
+    (property "Reference" "U202" (id 0) (at 106.045 76.9112 0)
       (effects (font (size 1.524 1.524)))
     )
@@
   (symbol (lib_id "Device:R_Pack04") (at 78.105 71.12 270) (mirror x)
     (in_bom yes) (on_board yes)
-    (property "Reference" "RN501" (id 0) (at 78.105 81.7118 90))
+    (property "Reference" "RN201" (id 0) (at 78.105 81.7118 90))
     (property "Value" "1k" (id 1) (at 78.105 79.4004 90))
     (property "Footprint" "Resistor_SMD:R_Array_Convex_4x0603" (id 2) (at 78.105 64.135 90)
@@
   (symbol (lib_id "Device:R_Pack04") (at 67.945 83.82 0)
     (in_bom yes) (on_board yes)
-    (property "Reference" "RN502" (id 0) (at 57.3532 83.82 90))
+    (property "Reference" "RN202" (id 0) (at 57.3532 83.82 90))
     (property "Value" "1k" (id 1) (at 59.6646 83.82 90))
     (property "Footprint" "Resistor_SMD:R_Array_Convex_4x0603" (id 2) (at 74.93 83.82 90)
@@
   (symbol (lib_id "power:GND") (at 62.865 88.9 0)
     (in_bom yes) (on_board yes)
-    (property "Reference" "#PWR0136" (id 0) (at 62.865 95.25 0)
+    (property "Reference" "#PWR0124" (id 0) (at 62.865 95.25 0)
       (effects (font (size 1.27 1.27)) hide)
     )
@@
   (symbol (lib_id "power:GND") (at 65.405 88.9 0)
     (in_bom yes) (on_board yes)
-    (property "Reference" "#PWR0137" (id 0) (at 65.405 95.25 0)
+    (property "Reference" "#PWR0125" (id 0) (at 65.405 95.25 0)
       (effects (font (size 1.27 1.27)) hide)
     )
@@
   (symbol (lib_id "power:GND") (at 67.945 88.9 0)
     (in_bom yes) (on_board yes)
-    (property "Reference" "#PWR0138" (id 0) (at 67.945 95.25 0)
+    (property "Reference" "#PWR0126" (id 0) (at 67.945 95.25 0)
       (effects (font (size 1.27 1.27)) hide)
     )
@@
   (symbol (lib_id "power:GND") (at 70.485 88.9 0)
     (in_bom yes) (on_board yes)
-    (property "Reference" "#PWR0139" (id 0) (at 70.485 95.25 0)
+    (property "Reference" "#PWR0127" (id 0) (at 70.485 95.25 0)
       (effects (font (size 1.27 1.27)) hide)
     )
@@
   (symbol (lib_id "power:GND") (at 112.395 69.215 0)
     (in_bom yes) (on_board yes)
-    (property "Reference" "#PWR0161" (id 0) (at 112.395 75.565 0)
+    (property "Reference" "#PWR0143" (id 0) (at 112.395 75.565 0)
       (effects (font (size 1.27 1.27)) hide)
     )
@@
   (symbol (lib_id "power:GND") (at 112.395 111.125 0)
     (in_bom yes) (on_board yes)
-    (property "Reference" "#PWR0166" (id 0) (at 112.395 117.475 0)
+    (property "Reference" "#PWR0148" (id 0) (at 112.395 117.475 0)
       (effects (font (size 1.27 1.27)) hide)
     )

Commit message: Packaged LS13-16 with the flyback diodes
Parts:
- renumbered RN201 to RN501, RN202 to RN502, U201 to U501, U202 to U502
Changed lines of the file:
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@@
   (symbol (lib_id "vnld5090:VNLD5090") (at 106.045 51.435 0)
     (in_bom yes) (on_board yes)
-    (property "Reference" "U201" (id 0) (at 106.045 35.0012 0)
+    (property "Reference" "U501" (id 0) (at 106.045 35.0012 0)
       (effects (font (size 1.524 1.524)))
     )
@@
   (symbol (lib_id "vnld5090:VNLD5090") (at 106.045 93.345 0)
     (in_bom yes) (on_board yes)
-    (property "Reference" "U202" (id 0) (at 106.045 76.9112 0)
+    (property "Reference" "U502" (id 0) (at 106.045 76.9112 0)
       (effects (font (size 1.524 1.524)))
     )
@@
   (symbol (lib_id "Device:R_Pack04") (at 78.105 71.12 270) (mirror x)
     (in_bom yes) (on_board yes)
-    (property "Reference" "RN201" (id 0) (at 78.105 81.7118 90))
+    (property "Reference" "RN501" (id 0) (at 78.105 81.7118 90))
     (property "Value" "1k" (id 1) (at 78.105 79.4004 90))
     (property "Footprint" "Resistor_SMD:R_Array_Convex_4x0603" (id 2) (at 78.105 64.135 90)
@@
   (symbol (lib_id "Device:R_Pack04") (at 67.945 83.82 0)
     (in_bom yes) (on_board yes)
-    (property "Reference" "RN202" (id 0) (at 57.3532 83.82 90))
+    (property "Reference" "RN502" (id 0) (at 57.3532 83.82 90))
     (property "Value" "1k" (id 1) (at 59.6646 83.82 90))
     (property "Footprint" "Resistor_SMD:R_Array_Convex_4x0603" (id 2) (at 74.93 83.82 90)

Commit message: Nearly finished routing
Parts:
- renumbered RN501 to RN201, RN502 to RN202, U501 to U201, U502 to U202
Changed lines of the file:
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@@
   (symbol (lib_id "vnld5090:VNLD5090") (at 106.045 51.435 0)
     (in_bom yes) (on_board yes)
-    (property "Reference" "U501" (id 0) (at 106.045 35.0012 0)
+    (property "Reference" "U201" (id 0) (at 106.045 35.0012 0)
       (effects (font (size 1.524 1.524)))
     )
@@
   (symbol (lib_id "vnld5090:VNLD5090") (at 106.045 93.345 0)
     (in_bom yes) (on_board yes)
-    (property "Reference" "U502" (id 0) (at 106.045 76.9112 0)
+    (property "Reference" "U202" (id 0) (at 106.045 76.9112 0)
       (effects (font (size 1.524 1.524)))
     )
@@
   (symbol (lib_id "Device:R_Pack04") (at 78.105 71.12 270) (mirror x)
     (in_bom yes) (on_board yes)
-    (property "Reference" "RN501" (id 0) (at 78.105 81.7118 90))
+    (property "Reference" "RN201" (id 0) (at 78.105 81.7118 90))
     (property "Value" "1k" (id 1) (at 78.105 79.4004 90))
     (property "Footprint" "Resistor_SMD:R_Array_Convex_4x0603" (id 2) (at 78.105 64.135 90)
@@
   (symbol (lib_id "Device:R_Pack04") (at 67.945 83.82 0)
     (in_bom yes) (on_board yes)
-    (property "Reference" "RN502" (id 0) (at 57.3532 83.82 90))
+    (property "Reference" "RN202" (id 0) (at 57.3532 83.82 90))
     (property "Value" "1k" (id 1) (at 59.6646 83.82 90))
     (property "Footprint" "Resistor_SMD:R_Array_Convex_4x0603" (id 2) (at 74.93 83.82 90)
