File: polygonus.kicad_sch (KiCad schematic)
At the start: 14 parts, among them J105 Conn_01x01, J107 Conn_01x01, J108 Conn_01x01, J3 Conn_01x32, J5 Conn_01x32, J6 Conn_01x16, J7 Conn_01x16

Commit message: Passing DRC
Connections:
- net GND: now also J7.5 (Pin_5), J7.6 (Pin_6), J7.7 (Pin_7), J7.8 (Pin_8)
Other:
- note removed: "Connectors 776228-1 776231-1 776231-2 Mating plugs 770680-1 776164-1 776164-2 Terminals 770854-1 all of the above cheap from ttiinc.com"
Changed lines of the file:
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@@
-    (effects (font (size 1.27 1.27)) (justify left bottom))
-  )
-  (text "Connectors\n776228-1\n\n776231-1\n\n776231-2\n\nMating plugs\n770680-1\n\n776164-1\n\n776164-2\n\nTerminals\n770854-1\n\nall of the above cheap from ttiinc.com"
-    (at 245.3694 132.9305 0)
     (effects (font (size 1.27 1.27)) (justify left bottom))
   )
@@
     (pin "1")
   )
-  (symbol (lib_id "power:GND") (at 273.05 39.37 270) (unit 1)
-    (in_bom yes) (on_board yes)
-    (property "Reference" "#PWR0140" (id 0) (at 266.7 39.37 0)
-      (effects (font (size 1.27 1.27)) hide)
-    )
-    (property "Value" "GND" (id 1) (at 269.7988 39.497 90)
-      (effects (font (size 1.27 1.27)) (justify right))
-    )
-    (property "Footprint" "" (id 2) (at 273.05 39.37 0)
-      (effects (font (size 1.27 1.27)) hide)
-    )
-    (property "Datasheet" "" (id 3) (at 273.05 39.37 0)
-      (effects (font (size 1.27 1.27)) hide)
-    )
-    (pin "1")
-  )
-  (symbol (lib_id "power:GND") (at 180.34 68.58 270) (unit 1)
-    (in_bom yes) (on_board yes)
-    (property "Reference" "#PWR0141" (id 0) (at 173.99 68.58 0)
-      (effects (font (size 1.27 1.27)) hide)
-    )
-    (property "Value" "GND" (id 1) (at 177.0888 68.707 90)
-      (effects (font (size 1.27 1.27)) (justify right))
-    )
-    (property "Footprint" "" (id 2) (at 180.34 68.58 0)
-      (effects (font (size 1.27 1.27)) hide)
-    )
-    (property "Datasheet" "" (id 3) (at 180.34 68.58 0)
+  (symbol (lib_id "power:GND") (at 273.2114 39.4319 270) (unit 1)
+    (in_bom yes) (on_board yes)
+    (property "Reference" "#PWR0140" (id 0) (at 266.8614 39.4319 0)
+      (effects (font (size 1.27 1.27)) hide)
+    )
+    (property "Value" "GND" (id 1) (at 269.9602 39.5589 90)
+      (effects (font (size 1.27 1.27)) (justify right))
+    )
+    (property "Footprint" "" (id 2) (at 273.2114 39.4319 0)
+      (effects (font (size 1.27 1.27)) hide)
+    )
+    (property "Datasheet" "" (id 3) (at 273.2114 39.4319 0)
       (effects (font (size 1.27 1.27)) hide)
     )
@@
     (pin "1")
   )
-  (symbol (lib_id "power:GND") (at 273.05 41.91 270) (unit 1)
-    (in_bom yes) (on_board yes)
-    (property "Reference" "#PWR0209" (id 0) (at 266.7 41.91 0)
-      (effects (font (size 1.27 1.27)) hide)
-    )
-    (property "Value" "GND" (id 1) (at 269.7988 42.037 90)
-      (effects (font (size 1.27 1.27)) (justify right))
-    )
-    (property "Footprint" "" (id 2) (at 273.05 41.91 0)
-      (effects (font (size 1.27 1.27)) hide)
-    )
-    (property "Datasheet" "" (id 3) (at 273.05 41.91 0)
-      (effects (font (size 1.27 1.27)) hide)
-    )
-    (pin "1")
-  )
-  (symbol (lib_id "power:GND") (at 273.05 34.29 270) (unit 1)
-    (in_bom yes) (on_board yes)
-    (property "Reference" "#PWR0112" (id 0) (at 266.7 34.29 0)
-      (effects (font (size 1.27 1.27)) hide)
-    )
-    (property "Value" "GND" (id 1) (at 269.7988 34.417 90)
-      (effects (font (size 1.27 1.27)) (justify right))
-    )
-    (property "Footprint" "" (id 2) (at 273.05 34.29 0)
-      (effects (font (size 1.27 1.27)) hide)
-    )
-    (property "Datasheet" "" (id 3) (at 273.05 34.29 0)
+  (symbol (lib_id "power:GND") (at 273.2114 41.9719 270) (unit 1)
+    (in_bom yes) (on_board yes)
+    (property "Reference" "#PWR0209" (id 0) (at 266.8614 41.9719 0)
+      (effects (font (size 1.27 1.27)) hide)
+    )
+    (property "Value" "GND" (id 1) (at 269.9602 42.0989 90)
+      (effects (font (size 1.27 1.27)) (justify right))
+    )
+    (property "Footprint" "" (id 2) (at 273.2114 41.9719 0)
+      (effects (font (size 1.27 1.27)) hide)
+    )
+    (property "Datasheet" "" (id 3) (at 273.2114 41.9719 0)
+      (effects (font (size 1.27 1.27)) hide)
+    )
+    (pin "1")
+  )
+  (symbol (lib_id "power:GND") (at 273.2114 34.3519 270) (unit 1)
+    (in_bom yes) (on_board yes)
+    (property "Reference" "#PWR0112" (id 0) (at 266.8614 34.3519 0)
+      (effects (font (size 1.27 1.27)) hide)
+    )
+    (property "Value" "GND" (id 1) (at 269.9602 34.4789 90)
+      (effects (font (size 1.27 1.27)) (justify right))
+    )
+    (property "Footprint" "" (id 2) (at 273.2114 34.3519 0)
+      (effects (font (size 1.27 1.27)) hide)
+    )
+    (property "Datasheet" "" (id 3) (at 273.2114 34.3519 0)
       (effects (font (size 1.27 1.27)) hide)
     )
@@
     (pin "1")
   )
-  (symbol (lib_id "power:GND") (at 273.05 36.83 270) (unit 1)
-    (in_bom yes) (on_board yes)
-    (property "Reference" "#PWR0107" (id 0) (at 266.7 36.83 0)
-      (effects (font (size 1.27 1.27)) hide)
-    )
-    (property "Value" "GND" (id 1) (at 269.7988 36.957 90)
-      (effects (font (size 1.27 1.27)) (justify right))
-    )
-    (property "Footprint" "" (id 2) (at 273.05 36.83 0)
-      (effects (font (size 1.27 1.27)) hide)
-    )
-    (property "Datasheet" "" (id 3) (at 273.05 36.83 0)
+  (symbol (lib_id "power:GND") (at 273.2114 36.8919 270) (unit 1)
+    (in_bom yes) (on_board yes)
+    (property "Reference" "#PWR0107" (id 0) (at 266.8614 36.8919 0)
+      (effects (font (size 1.27 1.27)) hide)
+    )
+    (property "Value" "GND" (id 1) (at 269.9602 37.0189 90)
+      (effects (font (size 1.27 1.27)) (justify right))
+    )
+    (property "Footprint" "" (id 2) (at 273.2114 36.8919 0)
+      (effects (font (size 1.27 1.27)) hide)
+    )
+    (property "Datasheet" "" (id 3) (at 273.2114 36.8919 0)
       (effects (font (size 1.27 1.27)) hide)
     )
@@
       (reference "#PWR0140") (unit 1) (value "GND") (footprint "")
     )
-    (path "/00000000-0000-0000-0000-00005d9f5241"
-      (reference "#PWR0141") (unit 1) (value "GND") (footprint "")
-    )
     (path "/00000000-0000-0000-0000-00005da12d1e"
