File: highside_quad.kicad_sch (KiCad schematic)
At the start: 14 parts, among them U40 BTS716G

Commit message: make hardware updates: - fix erc/drc errors - switch to VNLD5090 - switch to SOIC8 ignition drivers - BOM deduplication of similar parts
Parts:
- U40: LCSC (none) -> C85135
Changed lines of the file:
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@@
+      (effects (font (size 1.27 1.27)) hide)
+    )
+    (property "LCSC" "C85135" (at 67.31 71.12 0)
       (effects (font (size 1.27 1.27)) hide)
     )
