File: triggers.kicad_sch (KiCad schematic)
At the start: 39 parts, among them U10 SN74LVC2G17DB, U11 SRV05-4, U12 SRV05-4, U13 SRV05-4, U14 SN74LVC2G17DB, U8 SN74LVC2G17DB, U9 SN74LVC2G17DB

Commit message: make hardware updates: - fix erc/drc errors - switch to VNLD5090 - switch to SOIC8 ignition drivers - BOM deduplication of similar parts
Parts:
- U11, U12, U13: LCSC (none) -> C85364
Connections:
- net VR1+ renamed VR1
- net VR2+ renamed VR2
Changed lines of the file:
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@@
     (effects (font (size 1.27 1.27)) (justify left))
   )
-  (hierarchical_label "VR1+" (shape input) (at 209.55 29.1658 180) (fields_autoplaced)
+  (hierarchical_label "VR1" (shape input) (at 209.55 29.1658 180) (fields_autoplaced)
     (effects (font (size 1.27 1.27)) (justify right))
   )
@@
     (effects (font (size 1.27 1.27)) (justify left))
   )
-  (hierarchical_label "VR2+" (shape input) (at 208.28 91.44 180) (fields_autoplaced)
+  (hierarchical_label "VR2" (shape input) (at 208.28 91.44 180) (fields_autoplaced)
     (effects (font (size 1.27 1.27)) (justify right))
   )
@@
     )
     (property "Datasheet" "http://www.onsemi.com/pub/Collateral/SRV05-4-D.PDF" (at 142.875 71.755 0)
+      (effects (font (size 1.27 1.27)) hide)
+    )
+    (property "LCSC" "C85364" (at 142.875 71.755 0)
       (effects (font (size 1.27 1.27)) hide)
     )
@@
       (effects (font (size 1.27 1.27)) hide)
     )
+    (property "LCSC" "C85364" (at 127.635 164.465 0)
+      (effects (font (size 1.27 1.27)) hide)
+    )
     (pin "1")
     (pin "2")
@@
       (effects (font (size 1.27 1.27)) hide)
     )
+    (property "LCSC" "C85364" (at 237.49 62.23 0)
+      (effects (font (size 1.27 1.27)) hide)
+    )
