File: polygonus-Shortage-Version/ign4.kicad_sch (KiCad schematic)
At the start: 13 parts, among them U1701 MIC4427, U1702 MIC4427

Commit message: Switched highsides, changed TC4427 footprint, swapped USB to other side
Parts:
- U1602: renamed from U1701; footprint Package_SO:SOIC-8_3.9x4.9mm_P1.27mm -> Package_SO:MSOP-8_3x3mm_P0.65mm
- U1603: renamed from U1702; footprint Package_SO:SOIC-8_3.9x4.9mm_P1.27mm -> Package_SO:MSOP-8_3x3mm_P0.65mm
- renumbered C1701 to C1604, C1702 to C1605, C1703 to C1606, C1704 to C1607, C1705 to C1608, C1706 to C1609, R1701 to R1601, R1702 to R1602, R1703 to R1603, R1704 to R1604, RN1701 to RN1601
Changed lines of the file:
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@@
   (symbol (lib_id "Driver_FET:MIC4427") (at 76.835 46.99 0)
     (in_bom yes) (on_board yes)
-    (property "Reference" "U1701" (id 0) (at 80.01 55.88 0))
+    (property "Reference" "U1602" (id 0) (at 80.01 55.88 0))
     (property "Value" "MIC4427" (id 1) (at 81.28 38.1 0))
-    (property "Footprint" "Package_SO:SOIC-8_3.9x4.9mm_P1.27mm" (id 2) (at 76.835 54.61 0)
+    (property "Footprint" "Package_SO:MSOP-8_3x3mm_P0.65mm" (id 2) (at 76.835 54.61 0)
       (effects (font (size 1.27 1.27)) hide)
     )
@@
   (symbol (lib_id "Driver_FET:MIC4427") (at 76.835 85.09 0)
     (in_bom yes) (on_board yes)
-    (property "Reference" "U1702" (id 0) (at 80.01 93.98 0))
+    (property "Reference" "U1603" (id 0) (at 80.01 93.98 0))
     (property "Value" "MIC4427" (id 1) (at 81.28 76.2 0))
-    (property "Footprint" "Package_SO:SOIC-8_3.9x4.9mm_P1.27mm" (id 2) (at 76.835 92.71 0)
+    (property "Footprint" "Package_SO:MSOP-8_3x3mm_P0.65mm" (id 2) (at 76.835 92.71 0)
       (effects (font (size 1.27 1.27)) hide)
     )
@@
   (symbol (lib_id "Device:C_Small") (at 81.28 73.025 270)
     (in_bom yes) (on_board yes)
-    (property "Reference" "C1704" (id 0) (at 81.28 67.2084 90))
+    (property "Reference" "C1607" (id 0) (at 81.28 67.2084 90))
     (property "Value" "100n" (id 1) (at 81.28 69.5198 90))
     (property "Footprint" "Capacitor_SMD:C_0603_1608Metric" (id 2) (at 81.28 73.025 0)
@@
   (symbol (lib_id "power:GND") (at 76.835 57.15 0)
     (in_bom yes) (on_board yes)
-    (property "Reference" "#PWR0177" (id 0) (at 76.835 63.5 0)
+    (property "Reference" "#PWR0167" (id 0) (at 76.835 63.5 0)
       (effects (font (size 1.27 1.27)) hide)
     )
@@
   (symbol (lib_id "power:GND") (at 76.835 95.25 0)
     (in_bom yes) (on_board yes)
-    (property "Reference" "#PWR0178" (id 0) (at 76.835 101.6 0)
+    (property "Reference" "#PWR0168" (id 0) (at 76.835 101.6 0)
       (effects (font (size 1.27 1.27)) hide)
     )
@@
   (symbol (lib_id "Device:C_Small") (at 81.28 34.29 270)
     (in_bom yes) (on_board yes)
-    (property "Reference" "C1701" (id 0) (at 81.28 28.4734 90))
+    (property "Reference" "C1604" (id 0) (at 81.28 28.4734 90))
     (property "Value" "100n" (id 1) (at 81.28 30.7848 90))
     (property "Footprint" "Capacitor_SMD:C_0603_1608Metric" (id 2) (at 81.28 34.29 0)
@@
   (symbol (lib_id "power:+5V") (at 76.835 32.385 0)
     (in_bom yes) (on_board yes)
-    (property "Reference" "#PWR0179" (id 0) (at 76.835 36.195 0)
+    (property "Reference" "#PWR0169" (id 0) (at 76.835 36.195 0)
       (effects (font (size 1.27 1.27)) hide)
     )
@@
   (symbol (lib_id "power:+5V") (at 76.835 71.12 0)
     (in_bom yes) (on_board yes)
-    (property "Reference" "#PWR0180" (id 0) (at 76.835 74.93 0)
+    (property "Reference" "#PWR0170" (id 0) (at 76.835 74.93 0)
       (effects (font (size 1.27 1.27)) hide)
     )
@@
   (symbol (lib_id "power:GND") (at 83.82 73.025 90)
     (in_bom yes) (on_board yes)
-    (property "Reference" "#PWR0181" (id 0) (at 90.17 73.025 0)
+    (property "Reference" "#PWR0171" (id 0) (at 90.17 73.025 0)
       (effects (font (size 1.27 1.27)) hide)
     )
@@
   (symbol (lib_id "power:GND") (at 83.82 34.29 90)
     (in_bom yes) (on_board yes)
-    (property "Reference" "#PWR0182" (id 0) (at 90.17 34.29 0)
+    (property "Reference" "#PWR0172" (id 0) (at 90.17 34.29 0)
       (effects (font (size 1.27 1.27)) hide)
     )
@@
   (symbol (lib_id "Device:R") (at 93.98 44.45 270)
     (in_bom yes) (on_board yes)
-    (property "Reference" "R1701" (id 0) (at 93.98 42.545 90))
+    (property "Reference" "R1601" (id 0) (at 93.98 42.545 90))
     (property "Value" "100" (id 1) (at 93.98 44.45 90))
     (property "Footprint" "Resistor_SMD:R_0805_2012Metric" (id 2) (at 93.98 42.672 90)
@@
   (symbol (lib_id "Device:R") (at 93.98 49.53 270)
     (in_bom yes) (on_board yes)
-    (property "Reference" "R1702" (id 0) (at 93.98 47.625 90))
+    (property "Reference" "R1602" (id 0) (at 93.98 47.625 90))
     (property "Value" "100" (id 1) (at 93.98 49.53 90))
     (property "Footprint" "Resistor_SMD:R_0805_2012Metric" (id 2) (at 93.98 47.752 90)
@@
   (symbol (lib_id "Device:R") (at 93.98 82.55 270)
     (in_bom yes) (on_board yes)
-    (property "Reference" "R1703" (id 0) (at 93.98 80.645 90))
+    (property "Reference" "R1603" (id 0) (at 93.98 80.645 90))
     (property "Value" "100" (id 1) (at 93.98 82.55 90))
     (property "Footprint" "Resistor_SMD:R_0805_2012Metric" (id 2) (at 93.98 80.772 90)
@@
   (symbol (lib_id "Device:R") (at 93.98 87.63 270)
     (in_bom yes) (on_board yes)
-    (property "Reference" "R1704" (id 0) (at 93.98 85.725 90))
+    (property "Reference" "R1604" (id 0) (at 93.98 85.725 90))
     (property "Value" "100" (id 1) (at 93.98 87.63 90))
     (property "Footprint" "Resistor_SMD:R_0805_2012Metric" (id 2) (at 93.98 85.852 90)
@@
   (symbol (lib_id "Device:C") (at 99.695 55.245 0)
     (in_bom yes) (on_board yes)
-    (property "Reference" "C1703" (id 0) (at 102.616 54.0766 0)
+    (property "Reference" "C1606" (id 0) (at 102.616 54.0766 0)
       (effects (font (size 1.27 1.27)) (justify left))
     )
@@
   (symbol (lib_id "power:GND") (at 99.695 59.055 0)
     (in_bom yes) (on_board yes)
-    (property "Reference" "#PWR0183" (id 0) (at 99.695 65.405 0)
+    (property "Reference" "#PWR0173" (id 0) (at 99.695 65.405 0)
       (effects (font (size 1.27 1.27)) hide)
     )
@@
   (symbol (lib_id "Device:C") (at 99.695 38.735 180)
     (in_bom yes) (on_board yes)
-    (property "Reference" "C1702" (id 0) (at 102.616 37.5666 0)
+    (property "Reference" "C1605" (id 0) (at 102.616 37.5666 0)
       (effects (font (size 1.27 1.27)) (justify right))
     )
@@
   (symbol (lib_id "power:GND") (at 99.695 34.925 180)
     (in_bom yes) (on_board yes)
-    (property "Reference" "#PWR0184" (id 0) (at 99.695 28.575 0)
+    (property "Reference" "#PWR0174" (id 0) (at 99.695 28.575 0)
       (effects (font (size 1.27 1.27)) hide)
     )
@@
   (symbol (lib_id "Device:C") (at 99.695 76.835 180)
     (in_bom yes) (on_board yes)
-    (property "Reference" "C1705" (id 0) (at 102.616 75.6666 0)
+    (property "Reference" "C1608" (id 0) (at 102.616 75.6666 0)
       (effects (font (size 1.27 1.27)) (justify right))
     )
@@
   (symbol (lib_id "power:GND") (at 99.695 73.025 180)
     (in_bom yes) (on_board yes)
-    (property "Reference" "#PWR0185" (id 0) (at 99.695 66.675 0)
+    (property "Reference" "#PWR0175" (id 0) (at 99.695 66.675 0)
       (effects (font (size 1.27 1.27)) hide)
     )
@@
   (symbol (lib_id "Device:C") (at 99.695 93.345 0)
     (in_bom yes) (on_board yes)
-    (property "Reference" "C1706" (id 0) (at 102.616 92.1766 0)
+    (property "Reference" "C1609" (id 0) (at 102.616 92.1766 0)
       (effects (font (size 1.27 1.27)) (justify left))
     )
@@
   (symbol (lib_id "power:GND") (at 99.695 97.155 0)
     (in_bom yes) (on_board yes)
-    (property "Reference" "#PWR0186" (id 0) (at 99.695 103.505 0)
+    (property "Reference" "#PWR0176" (id 0) (at 99.695 103.505 0)
       (effects (font (size 1.27 1.27)) hide)
     )
@@
   (symbol (lib_id "Device:R_Pack04") (at 48.895 64.77 270)
     (in_bom yes) (on_board yes)
-    (property "Reference" "RN1701" (id 0) (at 50.0634 69.5452 0)
+    (property "Reference" "RN1601" (id 0) (at 50.0634 69.5452 0)
       (effects (font (size 1.27 1.27)) (justify left))
     )
@@
   (symbol (lib_id "power:GND") (at 43.815 67.31 270)
     (in_bom yes) (on_board yes)
-    (property "Reference" "#PWR0201" (id 0) (at 37.465 67.31 0)
+    (property "Reference" "#PWR0197" (id 0) (at 37.465 67.31 0)
       (effects (font (size 1.27 1.27)) hide)
     )
@@
   (symbol (lib_id "power:GND") (at 43.815 64.77 270)
     (in_bom yes) (on_board yes)
-    (property "Reference" "#PWR0202" (id 0) (at 37.465 64.77 0)
+    (property "Reference" "#PWR0198" (id 0) (at 37.465 64.77 0)
       (effects (font (size 1.27 1.27)) hide)
     )
@@
   (symbol (lib_id "power:GND") (at 43.815 62.23 270)
     (in_bom yes) (on_board yes)
-    (property "Reference" "#PWR0203" (id 0) (at 37.465 62.23 0)
+    (property "Reference" "#PWR0199" (id 0) (at 37.465 62.23 0)
       (effects (font (size 1.27 1.27)) hide)
     )
@@
   (symbol (lib_id "power:GND") (at 43.815 59.69 270)
     (in_bom yes) (on_board yes)
-    (property "Reference" "#PWR0204" (id 0) (at 37.465 59.69 0)
-      (effects (font (size 1.27 1.27)) hide)
-    )
+    (property "Reference" "#PWR0200" (id 0) (at 37.465 59.69 0)
+      (effects (font (size 1.27 1.27)) hide)
+    )

Commit message: Moved highsides about
Parts:
- renumbered C1604 to C1701, C1605 to C1702, C1606 to C1703, C1607 to C1704, C1608 to C1705, C1609 to C1706, R1601 to R1701, R1602 to R1702, R1603 to R1703, R1604 to R1704, RN1601 to RN1701, U1602 to U1701, U1603 to U1702
Changed lines of the file:
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@@
   (symbol (lib_id "Driver_FET:MIC4427") (at 76.835 46.99 0)
     (in_bom yes) (on_board yes)
-    (property "Reference" "U1602" (id 0) (at 80.01 55.88 0))
+    (property "Reference" "U1701" (id 0) (at 80.01 55.88 0))
     (property "Value" "MIC4427" (id 1) (at 81.28 38.1 0))
     (property "Footprint" "Package_SO:MSOP-8_3x3mm_P0.65mm" (id 2) (at 76.835 54.61 0)
@@
   (symbol (lib_id "Driver_FET:MIC4427") (at 76.835 85.09 0)
     (in_bom yes) (on_board yes)
-    (property "Reference" "U1603" (id 0) (at 80.01 93.98 0))
+    (property "Reference" "U1702" (id 0) (at 80.01 93.98 0))
     (property "Value" "MIC4427" (id 1) (at 81.28 76.2 0))
     (property "Footprint" "Package_SO:MSOP-8_3x3mm_P0.65mm" (id 2) (at 76.835 92.71 0)
@@
   (symbol (lib_id "Device:C_Small") (at 81.28 73.025 270)
     (in_bom yes) (on_board yes)
-    (property "Reference" "C1607" (id 0) (at 81.28 67.2084 90))
+    (property "Reference" "C1704" (id 0) (at 81.28 67.2084 90))
     (property "Value" "100n" (id 1) (at 81.28 69.5198 90))
     (property "Footprint" "Capacitor_SMD:C_0603_1608Metric" (id 2) (at 81.28 73.025 0)
@@
   (symbol (lib_id "power:GND") (at 76.835 57.15 0)
     (in_bom yes) (on_board yes)
-    (property "Reference" "#PWR0167" (id 0) (at 76.835 63.5 0)
+    (property "Reference" "#PWR0177" (id 0) (at 76.835 63.5 0)
       (effects (font (size 1.27 1.27)) hide)
     )
@@
   (symbol (lib_id "power:GND") (at 76.835 95.25 0)
     (in_bom yes) (on_board yes)
-    (property "Reference" "#PWR0168" (id 0) (at 76.835 101.6 0)
+    (property "Reference" "#PWR0178" (id 0) (at 76.835 101.6 0)
       (effects (font (size 1.27 1.27)) hide)
     )
@@
   (symbol (lib_id "Device:C_Small") (at 81.28 34.29 270)
     (in_bom yes) (on_board yes)
-    (property "Reference" "C1604" (id 0) (at 81.28 28.4734 90))
+    (property "Reference" "C1701" (id 0) (at 81.28 28.4734 90))
     (property "Value" "100n" (id 1) (at 81.28 30.7848 90))
     (property "Footprint" "Capacitor_SMD:C_0603_1608Metric" (id 2) (at 81.28 34.29 0)
@@
   (symbol (lib_id "power:+5V") (at 76.835 32.385 0)
     (in_bom yes) (on_board yes)
-    (property "Reference" "#PWR0169" (id 0) (at 76.835 36.195 0)
+    (property "Reference" "#PWR0179" (id 0) (at 76.835 36.195 0)
       (effects (font (size 1.27 1.27)) hide)
     )
@@
   (symbol (lib_id "power:+5V") (at 76.835 71.12 0)
     (in_bom yes) (on_board yes)
-    (property "Reference" "#PWR0170" (id 0) (at 76.835 74.93 0)
+    (property "Reference" "#PWR0180" (id 0) (at 76.835 74.93 0)
       (effects (font (size 1.27 1.27)) hide)
     )
@@
   (symbol (lib_id "power:GND") (at 83.82 73.025 90)
     (in_bom yes) (on_board yes)
-    (property "Reference" "#PWR0171" (id 0) (at 90.17 73.025 0)
+    (property "Reference" "#PWR0181" (id 0) (at 90.17 73.025 0)
       (effects (font (size 1.27 1.27)) hide)
     )
@@
   (symbol (lib_id "power:GND") (at 83.82 34.29 90)
     (in_bom yes) (on_board yes)
-    (property "Reference" "#PWR0172" (id 0) (at 90.17 34.29 0)
+    (property "Reference" "#PWR0182" (id 0) (at 90.17 34.29 0)
       (effects (font (size 1.27 1.27)) hide)
     )
@@
   (symbol (lib_id "Device:R") (at 93.98 44.45 270)
     (in_bom yes) (on_board yes)
-    (property "Reference" "R1601" (id 0) (at 93.98 42.545 90))
+    (property "Reference" "R1701" (id 0) (at 93.98 42.545 90))
     (property "Value" "100" (id 1) (at 93.98 44.45 90))
     (property "Footprint" "Resistor_SMD:R_0805_2012Metric" (id 2) (at 93.98 42.672 90)
@@
   (symbol (lib_id "Device:R") (at 93.98 49.53 270)
     (in_bom yes) (on_board yes)
-    (property "Reference" "R1602" (id 0) (at 93.98 47.625 90))
+    (property "Reference" "R1702" (id 0) (at 93.98 47.625 90))
     (property "Value" "100" (id 1) (at 93.98 49.53 90))
     (property "Footprint" "Resistor_SMD:R_0805_2012Metric" (id 2) (at 93.98 47.752 90)
@@
   (symbol (lib_id "Device:R") (at 93.98 82.55 270)
     (in_bom yes) (on_board yes)
-    (property "Reference" "R1603" (id 0) (at 93.98 80.645 90))
+    (property "Reference" "R1703" (id 0) (at 93.98 80.645 90))
     (property "Value" "100" (id 1) (at 93.98 82.55 90))
     (property "Footprint" "Resistor_SMD:R_0805_2012Metric" (id 2) (at 93.98 80.772 90)
@@
   (symbol (lib_id "Device:R") (at 93.98 87.63 270)
     (in_bom yes) (on_board yes)
-    (property "Reference" "R1604" (id 0) (at 93.98 85.725 90))
+    (property "Reference" "R1704" (id 0) (at 93.98 85.725 90))
     (property "Value" "100" (id 1) (at 93.98 87.63 90))
     (property "Footprint" "Resistor_SMD:R_0805_2012Metric" (id 2) (at 93.98 85.852 90)
@@
   (symbol (lib_id "Device:C") (at 99.695 55.245 0)
     (in_bom yes) (on_board yes)
-    (property "Reference" "C1606" (id 0) (at 102.616 54.0766 0)
+    (property "Reference" "C1703" (id 0) (at 102.616 54.0766 0)
       (effects (font (size 1.27 1.27)) (justify left))
     )
@@
   (symbol (lib_id "power:GND") (at 99.695 59.055 0)
     (in_bom yes) (on_board yes)
-    (property "Reference" "#PWR0173" (id 0) (at 99.695 65.405 0)
+    (property "Reference" "#PWR0183" (id 0) (at 99.695 65.405 0)
       (effects (font (size 1.27 1.27)) hide)
     )
@@
   (symbol (lib_id "Device:C") (at 99.695 38.735 180)
     (in_bom yes) (on_board yes)
-    (property "Reference" "C1605" (id 0) (at 102.616 37.5666 0)
+    (property "Reference" "C1702" (id 0) (at 102.616 37.5666 0)
       (effects (font (size 1.27 1.27)) (justify right))
     )
@@
   (symbol (lib_id "power:GND") (at 99.695 34.925 180)
     (in_bom yes) (on_board yes)
-    (property "Reference" "#PWR0174" (id 0) (at 99.695 28.575 0)
+    (property "Reference" "#PWR0184" (id 0) (at 99.695 28.575 0)
       (effects (font (size 1.27 1.27)) hide)
     )
@@
   (symbol (lib_id "Device:C") (at 99.695 76.835 180)
     (in_bom yes) (on_board yes)
-    (property "Reference" "C1608" (id 0) (at 102.616 75.6666 0)
+    (property "Reference" "C1705" (id 0) (at 102.616 75.6666 0)
       (effects (font (size 1.27 1.27)) (justify right))
     )
@@
   (symbol (lib_id "power:GND") (at 99.695 73.025 180)
     (in_bom yes) (on_board yes)
-    (property "Reference" "#PWR0175" (id 0) (at 99.695 66.675 0)
+    (property "Reference" "#PWR0185" (id 0) (at 99.695 66.675 0)
       (effects (font (size 1.27 1.27)) hide)
     )
@@
   (symbol (lib_id "Device:C") (at 99.695 93.345 0)
     (in_bom yes) (on_board yes)
-    (property "Reference" "C1609" (id 0) (at 102.616 92.1766 0)
+    (property "Reference" "C1706" (id 0) (at 102.616 92.1766 0)
       (effects (font (size 1.27 1.27)) (justify left))
     )
@@
   (symbol (lib_id "power:GND") (at 99.695 97.155 0)
     (in_bom yes) (on_board yes)
-    (property "Reference" "#PWR0176" (id 0) (at 99.695 103.505 0)
+    (property "Reference" "#PWR0186" (id 0) (at 99.695 103.505 0)
       (effects (font (size 1.27 1.27)) hide)
     )
@@
   (symbol (lib_id "Device:R_Pack04") (at 48.895 64.77 270)
     (in_bom yes) (on_board yes)
-    (property "Reference" "RN1601" (id 0) (at 50.0634 69.5452 0)
+    (property "Reference" "RN1701" (id 0) (at 50.0634 69.5452 0)
       (effects (font (size 1.27 1.27)) (justify left))
     )
@@
   (symbol (lib_id "power:GND") (at 43.815 67.31 270)
     (in_bom yes) (on_board yes)
-    (property "Reference" "#PWR0197" (id 0) (at 37.465 67.31 0)
+    (property "Reference" "#PWR0201" (id 0) (at 37.465 67.31 0)
       (effects (font (size 1.27 1.27)) hide)
     )
@@
   (symbol (lib_id "power:GND") (at 43.815 64.77 270)
     (in_bom yes) (on_board yes)
-    (property "Reference" "#PWR0198" (id 0) (at 37.465 64.77 0)
+    (property "Reference" "#PWR0202" (id 0) (at 37.465 64.77 0)
       (effects (font (size 1.27 1.27)) hide)
     )
@@
   (symbol (lib_id "power:GND") (at 43.815 62.23 270)
     (in_bom yes) (on_board yes)
-    (property "Reference" "#PWR0199" (id 0) (at 37.465 62.23 0)
+    (property "Reference" "#PWR0203" (id 0) (at 37.465 62.23 0)
       (effects (font (size 1.27 1.27)) hide)
     )
@@
   (symbol (lib_id "power:GND") (at 43.815 59.69 270)
     (in_bom yes) (on_board yes)
-    (property "Reference" "#PWR0200" (id 0) (at 37.465 59.69 0)
-      (effects (font (size 1.27 1.27)) hide)
-    )
+    (property "Reference" "#PWR0204" (id 0) (at 37.465 59.69 0)
+      (effects (font (size 1.27 1.27)) hide)
+    )

Commit message: clearout basic version
Other:
- company: rusEFI -> (none)
- title: rusEfi Proteus -> Polygonus
Changed lines of the file:
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@@
   (paper "A4")
   (title_block
-    (title "rusEfi Proteus")
-    (date "2022-04-09")
+    (title "Polygonus")
+    (date "2023-03-15")
     (rev "v0.7")
-    (company "rusEFI")
-    (comment 1 "github.com/mck1117/proteus")
     (comment 2 "rusefi.com/s/proteus")
   )
