File: polygonus-Shortage-Version/knock.kicad_sch (KiCad schematic)
At the start: 24 parts, among them U5 MCP6004

Commit message: clearout basic version
Other:
- company: rusEFI -> (none)
- title: rusEfi Proteus -> Polygonus
Changed lines of the file:
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@@
   (paper "A4")
   (title_block
-    (title "rusEfi Proteus")
-    (date "2022-04-09")
+    (title "Polygonus")
+    (date "2023-03-15")
     (rev "v0.7")
-    (company "rusEFI")
-    (comment 1 "github.com/mck1117/proteus")
     (comment 2 "rusefi.com/s/proteus")
   )

Commit message: Update to V1.3
Parts:
- renumbered C1903 to C15, C1901 to C16, C1902 to C17, C21 to C18, C22 to C19, C23 to C20, C24 to C21, C25 to C22, C26 to C23, R40 to R11, R38 to R12, R1901 to R13, R1902 to R14, R1903 to R15, R1904 to R16, R42 to R17, R43 to R18, R44 to R19, R45 to R20, R46 to R21, R47 to R22, U5 to U7
