File: polygonus-Shortage-Version/quad_analog.kicad_sch (KiCad schematic)
At the start: 24 parts, among them U3 SRV05-4, U901 MCP6004

Commit message: clearout basic version
Other:
- company: rusEFI -> (none)
- title: rusEfi Proteus -> Polygonus
Changed lines of the file:
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@@
   (paper "A4")
   (title_block
-    (title "rusEfi Proteus")
-    (date "2022-04-09")
+    (title "Polygonus")
+    (date "2023-03-15")
     (rev "v0.7")
-    (company "rusEFI")
-    (comment 1 "github.com/mck1117/proteus")
     (comment 2 "rusefi.com/s/proteus")
   )

Commit message: Update to V1.3
Parts:
- renumbered C901 to C56, C9 to C57, C10 to C58, C11 to C59, C12 to C60, R901 to R75, R902 to R76, R903 to R77, R904 to R78, R17 to R79, R18 to R80, R19 to R81, R20 to R82, R21 to R83, R22 to R84, R23 to R85, R24 to R86, RN901 to RN4, U901 to U21, U3 to U22
