File: polygonus-Shortage-Version/quad_analog_pullup.kicad_sch (KiCad schematic)
At the start: 21 parts, among them U1101 MCP6004, U4 SRV05-4

Commit message: clearout basic version
Other:
- company: rusEFI -> (none)
- title: rusEfi Proteus -> Polygonus
Changed lines of the file:
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@@
   (paper "A4")
   (title_block
-    (title "rusEfi Proteus")
-    (date "2022-04-09")
+    (title "Polygonus")
+    (date "2023-03-15")
     (rev "v0.7")
-    (company "rusEFI")
-    (comment 1 "github.com/mck1117/proteus")
     (comment 2 "rusefi.com/s/proteus")
   )

Commit message: Update to V1.3
Parts:
- renumbered C1101 to C40, C1409 to C41, C13 to C42, C14 to C43, C15 to C44, C16 to C45, R1101 to R39, R1102 to R40, R1103 to R41, R1104 to R42, R25 to R43, R26 to R44, R27 to R45, R28 to R46, R29 to R47, R30 to R48, R31 to R49, R32 to R50, RN1101 to RN1, U1101 to U15, U4 to U16
