File: polygonus-Shortage-Version/Keep_Alive.kicad_sch (KiCad schematic)
At the start: 7 parts, among them IC1 PSM712-LF-T7, U27 MIC5205-3.3YM5

Commit message: clearout basic version
Other:
- title: (none) -> Polygonus
Changed lines of the file:
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@@
 (kicad_sch (version 20211123) (generator eeschema)
   (paper "A4")
+  (title_block
+    (title "Polygonus")
+    (date "2023-03-15")
+    (rev "v0.7")
+  )
   (junction (at 105.41 76.2) (diameter 0) (color 0 0 0 0)
   )

Commit message: Update to V1.3
Parts:
- renumbered C32 to C89, C33 to C90, D5 to D16, D6 to D17, R54 to R107, U27 to U41
Changed lines of the file:
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@@
   (symbol (lib_id "power:GND") (at 105.41 87.63 0) (unit 1)
     (in_bom yes) (on_board yes) (fields_autoplaced)
-    (property "Reference" "#PWR07" (id 0) (at 105.41 93.98 0)
+    (property "Reference" "#PWR0258" (id 0) (at 105.41 93.98 0)
       (effects (font (size 1.27 1.27)) hide)
     )
@@
   (symbol (lib_id "Regulator_Linear:MIC5205-3.3YM5") (at 113.03 76.2 0) (unit 1)
     (in_bom yes) (on_board yes) (fields_autoplaced)
-    (property "Reference" "U27" (id 0) (at 113.03 66.04 0))
+    (property "Reference" "U41" (id 0) (at 113.03 66.04 0))
     (property "Value" "MIC5205-3.3YM5" (id 1) (at 113.03 68.58 0))
     (property "Footprint" "Package_TO_SOT_SMD:SOT-23-5" (id 2) (at 113.03 67.945 0)
@@
   (symbol (lib_id "power:GND") (at 127 78.74 0) (unit 1)
     (in_bom yes) (on_board yes) (fields_autoplaced)
-    (property "Reference" "#PWR09" (id 0) (at 127 85.09 0)
+    (property "Reference" "#PWR0260" (id 0) (at 127 85.09 0)
       (effects (font (size 1.27 1.27)) hide)
     )
@@
   (symbol (lib_id "power:GND") (at 90.17 107.95 0) (unit 1)
     (in_bom yes) (on_board yes) (fields_autoplaced)
-    (property "Reference" "#PWR06" (id 0) (at 90.17 114.3 0)
+    (property "Reference" "#PWR0257" (id 0) (at 90.17 114.3 0)
       (effects (font (size 1.27 1.27)) hide)
     )
@@
   (symbol (lib_id "Device:C_Small") (at 127 76.2 180) (unit 1)
     (in_bom yes) (on_board yes) (fields_autoplaced)
-    (property "Reference" "C33" (id 0) (at 129.54 74.9235 0)
+    (property "Reference" "C90" (id 0) (at 129.54 74.9235 0)
       (effects (font (size 1.27 1.27)) (justify right))
     )
@@
   (symbol (lib_id "Diode:1N4148WS") (at 139.7 73.66 180) (unit 1)
     (in_bom yes) (on_board yes) (fields_autoplaced)
-    (property "Reference" "D6" (id 0) (at 139.7 66.6485 0))
+    (property "Reference" "D17" (id 0) (at 139.7 66.6485 0))
     (property "Value" "1N4148WS" (id 1) (at 139.7 69.1885 0))
     (property "Footprint" "Diode_SMD:D_SOD-323" (id 2) (at 139.7 69.215 0)
@@
   (symbol (lib_id "power:GND") (at 113.03 83.82 0) (unit 1)
     (in_bom yes) (on_board yes) (fields_autoplaced)
-    (property "Reference" "#PWR08" (id 0) (at 113.03 90.17 0)
+    (property "Reference" "#PWR0259" (id 0) (at 113.03 90.17 0)
       (effects (font (size 1.27 1.27)) hide)
     )
@@
   (symbol (lib_id "Device:R_Small") (at 77.47 73.66 90) (unit 1)
     (in_bom yes) (on_board yes)
-    (property "Reference" "R54" (id 0) (at 77.47 76.2 90))
+    (property "Reference" "R107" (id 0) (at 77.47 76.2 90))
     (property "Value" "6.8k" (id 1) (at 77.47 78.74 90))
     (property "Footprint" "Resistor_SMD:R_0402_1005Metric" (id 2) (at 77.47 73.66 0)
@@
   (symbol (lib_id "Device:C_Small") (at 105.41 85.09 0) (unit 1)
     (in_bom yes) (on_board yes)
-    (property "Reference" "C32" (id 0) (at 100.33 80.01 0)
+    (property "Reference" "C89" (id 0) (at 100.33 80.01 0)
       (effects (font (size 1.27 1.27)) (justify left))
     )
@@
   (symbol (lib_id "Diode:1N4148WS") (at 71.12 73.66 180) (unit 1)
     (in_bom yes) (on_board yes) (fields_autoplaced)
-    (property "Reference" "D5" (id 0) (at 71.12 66.7482 0))
+    (property "Reference" "D16" (id 0) (at 71.12 66.7482 0))
     (property "Value" "1N4148WS" (id 1) (at 71.12 69.2882 0))
     (property "Footprint" "Diode_SMD:D_SOD-323" (id 2) (at 71.12 69.215 0)

Commit message: Fixed Caps. updated to V1.4
Parts:
- C89, C90: footprint Capacitor_SMD:C_0201_0603Metric -> Capacitor_SMD:C_0805_2012Metric
- R107: footprint Resistor_SMD:R_0402_1005Metric -> Resistor_SMD:R_0805_2012Metric
Changed lines of the file:
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@@
       (effects (font (size 1.27 1.27)) (justify right))
     )
-    (property "Footprint" "Capacitor_SMD:C_0201_0603Metric" (id 2) (at 127 76.2 0)
+    (property "Footprint" "Capacitor_SMD:C_0805_2012Metric" (id 2) (at 127 76.2 0)
       (effects (font (size 1.27 1.27)) hide)
     )
@@
     (property "Reference" "R107" (id 0) (at 77.47 76.2 90))
     (property "Value" "6.8k" (id 1) (at 77.47 78.74 90))
-    (property "Footprint" "Resistor_SMD:R_0402_1005Metric" (id 2) (at 77.47 73.66 0)
+    (property "Footprint" "Resistor_SMD:R_0805_2012Metric" (id 2) (at 77.47 73.66 0)
       (effects (font (size 1.27 1.27)) hide)
     )
@@
       (effects (font (size 1.27 1.27)) (justify left))
     )
-    (property "Footprint" "Capacitor_SMD:C_0201_0603Metric" (id 2) (at 105.41 85.09 0)
+    (property "Footprint" "Capacitor_SMD:C_0805_2012Metric" (id 2) (at 105.41 85.09 0)
       (effects (font (size 1.27 1.27)) hide)
     )
