File: polygonus-Shortage-Version/polygonus-Shortage-Version.kicad_sch (KiCad schematic)
At the start: 10 parts, among them J105 Conn_01x01, J107 Conn_01x01, J108 Conn_01x01, J3 Conn_01x32, J5 Conn_01x32, J6 Conn_01x16, J7 Conn_01x16

Commit message: Some silkscreen update
Connections:
- net 5V_SENSOR_1: no longer J3.7 (Pin_7)
- net 5V_SENSOR_2: no longer J3.6 (Pin_6)
- no-connect marks 0 -> 2
Changed lines of the file:
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@@
   (junction (at 194.31 102.87) (diameter 0) (color 0 0 0 0)
   )
+  (no_connect (at 227.33 36.83))
+  (no_connect (at 227.33 39.37))
   (wire (pts (xy 62.23 144.145) (xy 68.58 144.145))
     (stroke (width 0) (type default) (color 0 0 0 0))
@@
     (effects (font (size 1.27 1.27)) (justify right bottom))
   )
-  (label "5V_SENSOR_1" (at 227.33 39.37 180)
-    (effects (font (size 1.27 1.27)) (justify right bottom))
-  )
   (label "5V_SENSOR_1" (at 227.33 41.91 180)
     (effects (font (size 1.27 1.27)) (justify right bottom))
@@
   (label "LS10" (at 140.97 53.34 0)
     (effects (font (size 1.27 1.27)) (justify left bottom))
-  )
-  (label "5V_SENSOR_2" (at 227.33 36.83 180)
-    (effects (font (size 1.27 1.27)) (justify right bottom))
   )
   (label "LS6" (at 195.58 44.45 180)
@@
   )
   (symbol (lib_id "Connector_Generic:Conn_01x16") (at 278.2914 41.9719 0) (unit 1)
-    (in_bom yes) (on_board yes) (fields_autoplaced)
-    (property "Reference" "J7" (id 0) (at 280.8314 41.9718 0)
-      (effects (font (size 1.27 1.27)) (justify left))
-    )
-    (property "Value" "Conn_01x16" (id 1) (at 280.8314 44.5118 0)
-      (effects (font (size 1.27 1.27)) (justify left))
-    )
+    (in_bom yes) (on_board yes)
+    (property "Reference" "J7" (id 0) (at 259.9581 26.7811 0)
+      (effects (font (size 1.27 1.27)) (justify left))
+    )
+    (property "Value" "Conn_01x16" (id 1) (at 255.5749 29.9238 0)
+      (effects (font (size 1.27 1.27)) (justify left))
+    )

Commit message: clearout basic version
Other:
- company: rusEFI -> (none)
- title: rusEfi Proteus -> Polygonus
Changed lines of the file:
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@@
   (paper "A4")
   (title_block
-    (title "rusEfi Proteus")
-    (date "2022-04-09")
+    (title "Polygonus")
+    (date "2023-03-15")
     (rev "v0.7")
-    (company "rusEFI")
-    (comment 1 "github.com/mck1117/proteus")
-    (comment 2 "rusefi.com/s/proteus")
   )
   (junction (at 253.6325 75.2096) (diameter 0) (color 0 0 0 0)

Commit message: Update to V1.3
Parts:
- renumbered C17 to C1, F102 to F1, F101 to F2, J105 to J1, J107 to J2, J108 to J3, J5 to J4, J3 to J5
Connections:
- net RSVD: no longer J7.11 (Pin_11), J7.12 (Pin_12)
- new net RC1: J7.11 (Pin_11)
- new net RC2: J7.12 (Pin_12)
Other:
- sheet mcu ports: added RC1, RC2; removed none
